File: hw/jtag_switch.kicad_pcb (KiCad board)
At the start: 2 copper layers, 68.6 x 53.3 mm, 21 parts, among them J1 Digital/PWM, J2 Conn_ARM_JTAG_SWD_20, J3 Digital/PWM, J4 Conn_ARM_JTAG_SWD_20, J5 Conn_ARM_JTAG_SWD_20, J6 Power, J7 Analog, U1 TXS0108EPW, U2 TXS0108EPW

Commit message: HW v1.0 sent to Aisler
Parts:
- removed MH1, MH2, MH3, MH4: MountingHole_3.2mm, Arduino_MountingHole:MountingHole_3.2mm
- added C3: 100n, Capacitor_SMD:C_0603_1608Metric_Pad1.08x0.95mm_HandSolder, F.Cu at (129.1, 83.0)
- added C4: 100n, Capacitor_SMD:C_0603_1608Metric_Pad1.08x0.95mm_HandSolder, F.Cu at (126.9, 72.7)
- C1, C2: footprint Capacitor_SMD:C_0201_0603Metric -> Capacitor_SMD:C_0603_1608Metric_Pad1.08x0.95mm_HandSolder
- R1, R2, R3, R4: footprint Resistor_SMD:R_0201_0603Metric -> Resistor_SMD:R_0603_1608Metric_Pad0.98x0.95mm_HandSolder
- moved R4 39.2 mm to (158.3, 54.5), turned to 180 degrees
- moved R3 39.2 mm to (142.7, 54.5), turned to 180 degrees
- moved D1 38.6 mm to (138.5, 54.5), turned to 180 degrees
- moved D2 38.6 mm to (154.1, 54.5), turned to 180 degrees
- moved R2 4.62 mm to (130.9, 72.7)
- moved C1 2.89 mm to (125.0, 83.0), turned to 0 degrees
- moved U1 1.82 mm to (126.2, 78.2)
- moved C2 0.79 mm to (122.6, 72.7)
- moved R1 0.65 mm to (126.6, 62.8)
Connections:
- C1 pad 2: unconnected-(C1-Pad2) -> GND
Routing:
- net /*10: track 78.4 -> 40.3 mm, vias 2 -> 1
- net /*11: track 60.3 -> 33.9 mm
- net Net-(J2-VTREF): track 22.4 -> 28.1 mm
- net Net-(J4-VTREF): track 33.1 -> 36.9 mm
- net GND: track 3.74 -> 0.00 mm, vias 6 -> 5
- net Net-(J5-RTCK): track 22.4 -> 24.7 mm
- net Net-(J5-DBGRQ/NC): track 30.7 -> 33.0 mm
- net Net-(J5-TDO/SWO): track 23.9 -> 26.1 mm
- net Net-(J5-~{SRST}): track 26.3 -> 28.3 mm
- net Net-(J5-TCK/SWCLK): track 22.3 -> 23.9 mm
- net Net-(J2-TMS/SWDIO): track 10.8 -> 12.2 mm
- net Net-(J2-TDI): track 12.7 -> 14.0 mm
- net Net-(J2-~{TRST}): track 14.6 -> 15.8 mm
- net +3V3: track 48.0 -> 49.2 mm, vias 4 -> 2
- net Net-(J5-TMS/SWDIO): track 22.0 -> 23.1 mm
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Other:
- board text added: "DEBUGGER"
- board text added: "JTAG Switch"
- board text added: "TARGET 0"
- board text added: "TARGET 1"
- board text removed: "JTAG 0"
- board text removed: "JTAG 1"
