File: hw/jtag_switch.kicad_sch (KiCad schematic)
At the start: 17 parts, among them J1 Digital/PWM, J2 Conn_ARM_JTAG_SWD_20, J3 Digital/PWM, J4 Conn_ARM_JTAG_SWD_20, J5 Conn_ARM_JTAG_SWD_20, J6 Power, J7 Analog, U1 TXS0108EPW, U2 TXS0108EPW

Commit message: HW v1.0 sent to Aisler
Parts:
- added C3, C4: 100n, Capacitor_SMD:C_0603_1608Metric_Pad1.08x0.95mm_HandSolder, symbol Device:C
- C1, C2: footprint Capacitor_SMD:C_0201_0603Metric -> Capacitor_SMD:C_0603_1608Metric_Pad1.08x0.95mm_HandSolder
- R1, R2, R3, R4: footprint Resistor_SMD:R_0201_0603Metric -> Resistor_SMD:R_0603_1608Metric_Pad0.98x0.95mm_HandSolder
Connections:
- net GND: now also C1.2, C3.2, C4.1
- net at J4.1 (VTREF), U2.2 (VCCA): now also C4.2
- net at J2.1 (VTREF), U1.2 (VCCA): now also C3.1
